File: scoreboard.brd (EAGLE design)
At the start: 94 x 53.3 mm, 28 parts

Commit message: Updates from lastest user updates
Parts:
- removed BLUETOOTH: (no value), pinhead:1X08
- removed BUTTONS: (no value), pinhead:2X04
- removed D1, D2, D3, D4, D5, D6, D7, D8: 1N4004, adafruit:DO41-10
- removed R1, R2, R3, R4: (no value), adafruit:0805-THM
- removed RF-RECV: (no value), pinhead:1X07
- moved DISPLAY 49.3 mm to (17.8, 24.1), turned to 90 degrees
Connections:
- removed net N$1: D1.A, RF-RECV.2
- removed net N$19: BUTTONS.1, D5.A, R1.1
- removed net N$2: D2.A, RF-RECV.3
- removed net N$20: BUTTONS.3, D6.A, R2.1
- removed net N$21: BUTTONS.5, D7.A, R3.1
- removed net N$22: BUTTONS.7, D8.A, R4.1
- removed net N$3: D3.A, RF-RECV.4
- removed net N$4: D4.A, RF-RECV.5
- net +5V: no longer BLUETOOTH.5, BUTTONS.2, BUTTONS.4, BUTTONS.6, BUTTONS.8, RF-RECV.6
- net DIG36: no longer D1.C, D5.C
- net DIG37: no longer D2.C, D6.C
- net DIG38: no longer D3.C, D7.C
- net DIG39: no longer D4.C, D8.C
- net GND: no longer BLUETOOTH.2, BLUETOOTH.7, R1.2, R2.2, R3.2, R4.2, RF-RECV.7
- net RX1_D19: no longer BLUETOOTH.3
- net TX1_D18: no longer BLUETOOTH.4
Routing:
- net DIG36: track 84.3 -> 0.00 mm
- net DIG37: track 80.4 -> 0.00 mm
- net DIG50: track 88.5 -> 15.8 mm, vias 1 -> 0
- net DIG38: track 72.4 -> 0.00 mm
- net DIG39: track 69.4 -> 0.00 mm
- net DIG26: track 79.6 -> 14.6 mm
- net DIG51: track 78.5 -> 18.1 mm, vias 1 -> 0
- net DIG24: track 73.1 -> 14.6 mm
- net GND: track 202.0 -> 144.9 mm
- net DIG25: track 71.1 -> 14.6 mm
- net DIG28: track 65.7 -> 12.0 mm
- net N$19: track 53.3 -> 0.00 mm
- net DIG27: track 71.0 -> 18.2 mm
- net +5V: track 130.7 -> 78.4 mm, vias 2 -> 0
- net N$20: track 50.6 -> 0.00 mm
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Other:
- board text added: "<--- R1"
