File: scoreboard.sch (EAGLE design)
At the start: 28 parts

Commit message: Updates from lastest user updates
Parts:
- removed BLUETOOTH: (no value), pinhead:PINHD-1X8
- removed BUTTONS: (no value), pinhead:PINHD-2X4
- removed D1, D2, D3, D4, D5, D6, D7, D8: 1N4004, adafruit:1N4004
- removed R1, R2, R3, R4: (no value), adafruit:FLIPFLOP-RES
- removed RF-RECV: (no value), pinhead:PINHD-1X7
Connections:
- removed net N$1: D1.A, RF-RECV.2
- removed net N$19: BUTTONS.1, D5.A, R1.1
- removed net N$2: D2.A, RF-RECV.3
- removed net N$20: BUTTONS.3, D6.A, R2.1
- removed net N$21: BUTTONS.5, D7.A, R3.1
- removed net N$22: BUTTONS.7, D8.A, R4.1
- removed net N$3: D3.A, RF-RECV.4
- removed net N$4: D4.A, RF-RECV.5
- net +5V: no longer BLUETOOTH.5, BUTTONS.2, BUTTONS.4, BUTTONS.6, BUTTONS.8, RF-RECV.6
- net DIG36: no longer D1.C, D5.C
- net DIG37: no longer D2.C, D6.C
- net DIG38: no longer D3.C, D7.C
- net DIG39: no longer D4.C, D8.C
- net GND: no longer BLUETOOTH.2, BLUETOOTH.7, R1.2, R2.2, R3.2, R4.2, RF-RECV.7
- net RX1_D19: no longer BLUETOOTH.3
- net TX1_D18: no longer BLUETOOTH.4
